Commit message: Scene: blue plates on a 12.5 mm aluminium fixture plate; fixture/trolley collision boxes
- Lab photos: robot base on the trolley top; blue plates on a slotted aluminium
  plate on the same top. Plate undersides now z = 12.5 mm (thickness from the
  ur3_lfd trolley mesh, to be measured on the real plate).
- compute_scene_registration: --fixture-thickness; generates fixture_plate and
  trolley_top box STLs (cad/environment), added to scene_model, MoveIt
  (OBJECT_IDS) and the RViz scene URDF (replaces the visual patch).
- Re-ran scene validation, Stage 8 (A/B1/B2/B2R) and Stage 9 offline: all
  outcomes unchanged; numbers shift slightly (grasp 12.5 mm shorter along a
  2.6 deg tilted tool axis): arrival offset 2.60 -> 2.03 mm, B2 gap 0.286 ->
  0.258 mm, B2R ring contact gone. New references kept beside the z = 0 ones.

Co-Authored-By: Claude Opus 5.5 <noreply@anthropic.com>
Claude-Session: https://claude.ai/code/session_0121fGeGCexoSeqbVFvLJFuv

File: urdf/variant_scene.urdf.xacro (robot description, xacro)
@@ -20,5 +20,4 @@
   <material name="part_blue"><color rgba="0.20 0.40 1.00 1.0"/></material>
   <material name="fitting_blue"><color rgba="0.12 0.30 0.90 1.0"/></material>
-  <material name="surface_grey"><color rgba="0.75 0.75 0.78 0.35"/></material>
   <!-- Root = robot base frame (provided by the UR3e robot_state_publisher) -->
   <link name="base"/>
@@ -68,17 +67,27 @@
   </xacro:macro>
   <xacro:variants i="1"/>
-  <!-- ===== Visual-only trolley-top patch (shows the assumed surface height) ===== -->
-  <link name="trolley_surface_patch">
-    <visual>
-      <geometry><box size="${reg['trolley_patch']['size_m'][0]} ${reg['trolley_patch']['size_m'][1]} ${reg['trolley_patch']['size_m'][2]}"/></geometry>
-      <material name="surface_grey"/>
-    </visual>
-  </link>
-  <joint name="trolley_surface_patch_joint" type="fixed">
-    <parent link="base"/>
-    <child link="trolley_surface_patch"/>
-    <origin xyz="${reg['trolley_patch']['xyz_m'][0]} ${reg['trolley_patch']['xyz_m'][1]} ${reg['trolley_patch']['xyz_m'][2]}"
-            rpy="0 0 ${reg['trolley_patch']['yaw_rad']}"/>
-  </joint>
+  <!-- ===== Environment collision boxes (aluminium fixture plate, trolley top) =====
+       Boxes generated by compute_scene_registration.py (cad/environment/*.stl, mm). -->
+  <material name="aluminium"><color rgba="0.78 0.79 0.82 1.0"/></material>
+  <material name="trolley_dark"><color rgba="0.15 0.15 0.16 1.0"/></material>
+  <xacro:macro name="env_box" params="name material">
+    <link name="${name}">
+      <visual>
+        <geometry><mesh filename="package://${pkg}/cad/environment/${name}.stl" scale="${mm} ${mm} ${mm}"/></geometry>
+        <material name="${material}"/>
+      </visual>
+      <collision>
+        <geometry><mesh filename="package://${pkg}/cad/environment/${name}.stl" scale="${mm} ${mm} ${mm}"/></geometry>
+      </collision>
+    </link>
+    <joint name="${name}_joint" type="fixed">
+      <parent link="base"/>
+      <child link="${name}"/>
+      <origin xyz="${reg['environment'][name]['xyz_m'][0]} ${reg['environment'][name]['xyz_m'][1]} ${reg['environment'][name]['xyz_m'][2]}"
+              rpy="0 0 ${reg['environment'][name]['yaw_rad']}"/>
+    </joint>
+  </xacro:macro>
+  <xacro:env_box name="fixture_plate" material="aluminium"/>
+  <xacro:env_box name="trolley_top" material="trolley_dark"/>
   <!-- ===== Optional: existing trolley mesh from ur3_lfd (read-only reference) =====
        Pose in `base` composed from ur3_lfd/urdf/trolley.urdf.xacro (base_link is Rz(pi) from base):
